File: _autosave-pcb1.kicad_pcb (KiCad board)
At the start: 2 copper layers, 49.5 x 49.5 mm, 68 parts, among them P1 CONN_01X06, P10 M1, P11 M2, P12 CONN_01X02, P2 CONN_01X06, P3 CONN_01X06, P4 CONN_01X06, P5 UART, P6 SWD, Q1 IRF9540N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

Commit message: almoast half ready ;)
Parts:
- moved C4 17.1 mm to (205.1, 73.7)
- moved C15 13.3 mm to (205.1, 71.8)
- moved C16 12.3 mm to (209.6, 66.0)
- moved C17 12.3 mm to (209.6, 64.1)
- moved R10 12.2 mm to (215.3, 62.2), turned to 270 degrees
- moved R6 1.42 mm to (215.3, 65.4), turned to 270 degrees
Changed lines of the file:
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@@
   )
   (module Capacitors_SMD:C_0805 (layer F.Cu)
-    (at 205.105 56.515 180)
+    (at 205.105 73.66 180)
     (descr "Capacitor SMD 0805, reflow soldering, AVX (see smccp.pdf)")
     (tags "capacitor 0805")
@@
   )
   (module Capacitors_SMD:C_0805 (layer F.Cu)
-    (at 205.105 58.42 180)
+    (at 205.105 71.755 180)
     (descr "Capacitor SMD 0805, reflow soldering, AVX (see smccp.pdf)")
     (tags "capacitor 0805")
@@
   )
   (module Capacitors_SMD:C_0805 (layer F.Cu)
-    (at 205.105 54.61 180)
+    (at 209.55 66.04 180)
     (descr "Capacitor SMD 0805, reflow soldering, AVX (see smccp.pdf)")
     (tags "capacitor 0805")
@@
   )
   (module Capacitors_SMD:C_0805 (layer F.Cu)
-    (at 205.105 52.705 180)
+    (at 209.55 64.135 180)
     (descr "Capacitor SMD 0805, reflow soldering, AVX (see smccp.pdf)")
     (tags "capacitor 0805")
@@
   )
   (module Resistors_SMD:R_0805 (layer F.Cu)
-    (at 214.63 66.675 180)
+    (at 215.265 65.405 270)
     (descr "Resistor SMD 0805, reflow soldering, Vishay (see dcrcw.pdf)")
     (tags "resistor 0805")
     (attr smd)
-    (fp_text reference R6 (at 0 -1.65 180) (layer F.SilkS)
-      (effects (font (size 1 1) (thickness 0.15)))
-    )
-    (fp_text value 510R (at 0 1.75 180) (layer F.Fab)
-      (effects (font (size 1 1) (thickness 0.15)))
-    )
-    (fp_text user %R (at 0 -1.65 180) (layer F.Fab)
+    (fp_text reference R6 (at 0 -1.65 270) (layer F.SilkS)
+      (effects (font (size 1 1) (thickness 0.15)))
+    )
+    (fp_text value 510R (at 0 1.75 270) (layer F.Fab)
+      (effects (font (size 1 1) (thickness 0.15)))
+    )
+    (fp_text user %R (at 0 -1.65 270) (layer F.Fab)
       (effects (font (size 1 1) (thickness 0.15)))
     )
@@
     (fp_line (start 1.55 0.9) (end 1.55 -0.9) (layer F.CrtYd) (width 0.05))
     (fp_line (start 1.55 0.9) (end -1.55 0.9) (layer F.CrtYd) (width 0.05))
-    (pad 1 smd rect (at -0.95 0 180) (size 0.7 1.3) (layers F.Cu F.Paste F.Mask)
+    (pad 1 smd rect (at -0.95 0 270) (size 0.7 1.3) (layers F.Cu F.Paste F.Mask)
       (net 63 "Net-(R10-Pad2)"))
-    (pad 2 smd rect (at 0.95 0 180) (size 0.7 1.3) (layers F.Cu F.Paste F.Mask)
+    (pad 2 smd rect (at 0.95 0 270) (size 0.7 1.3) (layers F.Cu F.Paste F.Mask)
       (net 1 GND))
     (model Resistors_SMD.3dshapes/R_0805.wrl
@@
   )
   (module Resistors_SMD:R_0805 (layer F.Cu)
-    (at 226.06 67.945)
+    (at 215.265 62.23 270)
     (descr "Resistor SMD 0805, reflow soldering, Vishay (see dcrcw.pdf)")
     (tags "resistor 0805")
     (attr smd)
-    (fp_text reference R10 (at 0 -1.65) (layer F.SilkS)
-      (effects (font (size 1 1) (thickness 0.15)))
-    )
-    (fp_text value 10k (at 0 1.75) (layer F.Fab)
-      (effects (font (size 1 1) (thickness 0.15)))
-    )
-    (fp_text user %R (at 0 -1.65) (layer F.Fab)
+    (fp_text reference R10 (at 0 -1.65 270) (layer F.SilkS)
+      (effects (font (size 1 1) (thickness 0.15)))
+    )
+    (fp_text value 10k (at 0 1.75 270) (layer F.Fab)
+      (effects (font (size 1 1) (thickness 0.15)))
+    )
+    (fp_text user %R (at 0 -1.65 270) (layer F.Fab)
       (effects (font (size 1 1) (thickness 0.15)))
     )
@@
     (fp_line (start 1.55 0.9) (end 1.55 -0.9) (layer F.CrtYd) (width 0.05))
     (fp_line (start 1.55 0.9) (end -1.55 0.9) (layer F.CrtYd) (width 0.05))
-    (pad 1 smd rect (at -0.95 0) (size 0.7 1.3) (layers F.Cu F.Paste F.Mask)
+    (pad 1 smd rect (at -0.95 0 270) (size 0.7 1.3) (layers F.Cu F.Paste F.Mask)
       (net 2 +3V3))
-    (pad 2 smd rect (at 0.95 0) (size 0.7 1.3) (layers F.Cu F.Paste F.Mask)
+    (pad 2 smd rect (at 0.95 0 270) (size 0.7 1.3) (layers F.Cu F.Paste F.Mask)
       (net 63 "Net-(R10-Pad2)"))
     (model Resistors_SMD.3dshapes/R_0805.wrl
