File: pcb1.sch (KiCad schematic (older format))
At the start: 53 parts, among them P1 Vss, Rx,Tx, Vee, P2 M1 A, P3 M1 B, P4 M2 A, P5 M2 B, P6 encoder 1, P7 encoder 2, Q1 IRF9540N, U1 LM7812, U2 STM32F030C6Tx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

Commit message: almoast half ready ;)
Parts:
- removed C1, C3: 0.33u, Capacitors_SMD:C_1210, symbol CP1
- removed C13: 100n, symbol C
- removed C2, C4: 0.1u, Capacitors_SMD:C_1210, symbol CP1
- removed D2, D3, D5, D6, D7, D8, D9: D, Diodes_THT:D_T-1_P5.08mm_Horizontal, symbol D
- removed P2: M1 A, Connectors:PINTST, symbol CONN_01X01
- removed P3: M1 B, Connectors:PINTST, symbol CONN_01X01
- removed P4: M2 A, Connectors:PINTST, symbol CONN_01X01
- removed P5: M2 B, Connectors:PINTST, symbol CONN_01X01
- removed P6: encoder 1, symbol CONN_01X12
- removed P7: encoder 2, symbol CONN_01X12
- removed R1, R? (x2): R, symbol R
- removed U1: LM7812, TO_SOT_Packages_THT:TO-220_Vertical, symbol LM7812
- removed U3: 7805, TO_SOT_Packages_THT:TO-220_Vertical, symbol 7805
- removed U5, U6: HL293D, MyLib:HL293D, symbol HL293D
- removed U? (x2): 74AHC1G14, symbol 74AHC1G14
- added C15, C17, C18, C6, C8: 1u, Capacitors_SMD:C_0805, symbol C
- added C16, C2, C20, C21, C22, C25, C26, C29, C30, C31, C4, C7: 100n, Capacitors_SMD:C_0805, symbol C
- added C19: 10u, Capacitors_SMD:C_0805, symbol C
- added C23, C27: 0.33u, Capacitors_SMD:C_0805, symbol CP
- added C24, C28: 0.1u, Capacitors_SMD:C_0805, symbol CP
- added F1: Polyfuse, SparkFun:SparkFun-PTC-1206, symbol Polyfuse
- added P1, P2, P3, P4: CONN_01X06, Connectors:PINHEAD1-6, symbol CONN_01X06
- added P10: M1, Connectors:bornier2, symbol CONN_01X02
- added P11: M2, Connectors:bornier2, symbol CONN_01X02
- added P12: CONN_01X02, Connectors:bornier2, symbol CONN_01X02
- added P6: SWD, SparkFun:SparkFun-1X04, symbol CONN_01X04
- added R10, R11, R7: 10k, Resistors_SMD:R_0805, symbol R
- added R3, R4: 100k, Resistors_SMD:R_0805, symbol R
- added U1, U5: 74AHC1G14, TO_SOT_Packages_SMD:SOT-353_SC-70-5, symbol 74AHC1G14
- added U10, U9: HL293D, Housings_SOIC:SOIC-20W_7.5x12.8mm_Pitch1.27mm, symbol HL293D
- added U4: LM7812CT, Power_Integrations:TO-220, symbol LM7812CT
- added U7: LM7805CT, TO_SOT_Packages_SMD:SOT-223-3Lead_TabPin2, symbol LM7805CT
- C1: renamed from C11; footprint (none) -> Capacitors_SMD:C_0805
- C10: renamed from C6; footprint Discret:CP5 -> Capacitors_SMD:C_0805
- C11: renamed from C7; footprint Capacitors_THT:C_Disc_D3.0mm_W1.6mm_P2.50mm -> Capacitors_SMD:C_0805
- C12: renamed from C8; footprint Capacitors_THT:C_Disc_D3.0mm_W1.6mm_P2.50mm -> Capacitors_SMD:C_0805
- C13: renamed from C9; footprint Capacitors_THT:C_Disc_D3.0mm_W1.6mm_P2.50mm -> Capacitors_SMD:C_0805
- C14: renamed from C10; footprint Capacitors_THT:C_Disc_D3.0mm_W1.6mm_P2.50mm -> Capacitors_SMD:C_0805
- C3: renamed from C12; footprint (none) -> Capacitors_SMD:C_0805
- C5: renamed from C14; value 4.7u -> 1u; footprint (none) -> Capacitors_SMD:C_0805
- C9: renamed from C?; footprint Discret:CP5 -> Capacitors_SMD:C_0805
- D1: renamed from D10; footprint (none) -> Diodes_SMD:D_0805
- D2: renamed from D11; footprint (none) -> Diodes_SMD:D_0805
- D3: renamed from D12; footprint (none) -> Diodes_SMD:D_0805
- D4: footprint Diodes_THT:D_T-1_P5.08mm_Horizontal -> Diodes_SMD:D_0805
- P5: renamed from P1; value Vss, Rx,Tx, Vee -> UART; footprint (none) -> SparkFun:SparkFun-1X04
- Q1: footprint Power_Integrations:TO-220 -> TO_SOT_Packages_THT:TO-220_Vertical
- R1: renamed from R3; value R -> 100R; footprint (none) -> Resistors_SMD:R_0805
- R2: renamed from R4; value 1k -> 10k; footprint (none) -> Resistors_SMD:R_0805
- R5: renamed from R?; footprint (none) -> Resistors_SMD:R_0805
- R6: renamed from R5; value 10k -> 510R; footprint (none) -> Resistors_SMD:R_0805
- R8: renamed from R?; value R -> 10k; footprint (none) -> Resistors_SMD:R_0805
- R9: renamed from R2; value R -> 100R; footprint (none) -> Resistors_SMD:R_0805
- S1: footprint SparkFun:SparkFun-REED_SWITCH_PTH -> Buttons_Switches_SMD:SW_SPST_TL3342
- U2: renamed from U8; footprint MFSOP-6 -> Buttons_Switches_SMD:SW_DIP_x2_W6.15mm_Slide_Omron_A6H; symbol LTV-358T -> LTV-358T-RESCUE-pcb1
- U3: renamed from U?; footprint MFSOP-6 -> Buttons_Switches_SMD:SW_DIP_x2_W6.15mm_Slide_Omron_A6H; symbol LTV-358T -> LTV-358T-RESCUE-pcb1
- U8: renamed from U?; footprint (none) -> TO_SOT_Packages_SMD:SOT-223; symbol LM1117-3.3 -> LM1117-3.3-RESCUE-pcb1
- renumbered U2 to U6
Connections:
- net labels added: +3V3, +5C, Enc0, Enc1, Enc2, Enc3, IntRx, IntTx, SWCLK
- net labels removed: 12V, 3.3V, 5V, SWDCLK, Vdd, Vss
- wire segments 173 -> 301
- no-connect marks 59 -> 10
Other:
- note added: "Kondensatory filtrujące przy zasilaniu procesora"
- note added: "Przycisk reset oraz\nPuDwn R do BOOT0"
- note added: "ST Link (SWD)"
- note added: "Stablilizatory 12->5->3.3 z filatracją oraz diodami zapobiegającymi szplikom"
- note added: "Uart z optoizolacją"
- note added: "Wejścia z encoderów"
- note added: "Zanezpieczenie przed\n odwrotną polaryzacją"
- note added: "Zasilanie płytki 24V"
- note removed: "Stablilizatory 12->5->3.3 z filatracją"
- note removed: "Zanezpieczenie przed odwrotną polaryzacją"
- note removed: "silnki: PA6 (TIM2 CH1) - M1 PWM, PA4, PA5 (GPIO)\n PA7 (TIM2 CH2) - M2 PWM, PA8, PA9 (GPIO) \nuart: PA2, PA3 (USART1)\nenkodery: ???\n"
- moved on the sheet: C1, C10, C11, C12, C13, C14, C3, C5, C9, D1, D2, D3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

Commit message: 5x5
Parts:
- removed P6: SWD, SparkFun:SparkFun-1X04, symbol CONN_01X04
- removed R3, R4: 100k, Resistors_SMD:R_0805, symbol R
- removed U6: STM32F030C6Tx, Housings_QFP:LQFP-48_7x7mm_Pitch0.5mm, symbol STM32F030C6Tx
- added P6: CONN_01X05, SparkFun:SparkFun-1X05-1.27MM, symbol CONN_01X05
- added U6: STM32F103C6Tx, Housings_QFP:LQFP-48_7x7mm_Pitch0.5mm, symbol STM32F103C6Tx
Connections:
- net +3V3: now also U6.24 (VDD), U6.36 (VDD), U6.48 (VDD)
- net Enc0: now also U6.10 (ADC1_IN0/ADC2_IN0/SYS_WKUP/TIM2_CH1/TIM2_ETR/USART2_CTS/PA0), U6.2 (PC13/RTC_OUT/RTC_TAMPER)
- net Enc1: now also U6.11 (ADC1_IN1/ADC2_IN1/TIM2_CH2/USART2_RTS/PA1), U6.3 (PC14/RCC_OSC32_IN)
- net Enc2: now also U6.4 (PC15/ADC1_EXTI15/ADC2_EXTI15/RCC_OSC32_OUT)
- net Enc3: now also U6.33 (CAN_TX/TIM1_ETR/USART1_RTS/USB_DP/PA12)
- net GND: now also P6.1 (P1), U6.23 (VSS), U6.35 (VSS), U6.47 (VSS), U6.8 (VSSA)
- net IntRx: now also U6.12 (ADC1_IN2/ADC2_IN2/TIM2_CH3/USART2_TX/PA2)
- net IntTx: now also U6.13 (ADC1_IN3/ADC2_IN3/TIM2_CH4/USART2_RX/PA3)
- net SWCLK: now also P6.3 (P3), U6.37 (SYS_JTCK-SWCLK/PA14)
- net SWDIO: now also P6.4 (P4), U6.34 (SYS_JTMS-SWDIO/PA13)
- net at U9.12 (3A), U9.2 (1A): now also U6.14 (ADC1_IN4/ADC2_IN4/SPI1_NSS/USART2_CK/PA4)
- net at U9.19 (4A), U9.9 (2A): now also U6.15 (ADC1_IN5/ADC2_IN5/SPI1_SCK/PA5)
- net at U9.1 (1,2EN), U9.11 (3,4_EN): now also U6.16 (ADC1_IN6/ADC2_IN6/SPI1_MISO/TIM1_BKIN/TIM3_CH1/PA6)
- net at P1.4 (P4): now also U6.18 (PB0/ADC1_IN8/ADC2_IN8/TIM1_CH2N/TIM3_CH3)
- net at P1.3 (P3): now also U6.19 (PB1/ADC1_IN9/ADC2_IN9/TIM1_CH3N/TIM3_CH4)
- net at P1.2 (P2): now also U6.20 (PB2/BOOT1)
- net at P3.4 (P4): now also U6.22 (PB11/ADC1_EXTI11/ADC2_EXTI11/TIM2_CH4)
- net at P3.3 (P3): now also U6.25 (PB12/TIM1_BKIN)
- net at P3.2 (P2): now also U6.26 (PB13/TIM1_CH1N)
- net at P3.1 (P1): now also U6.27 (PB14/TIM1_CH2N)
- net at P4.6 (P6): now also U6.28 (PB15/ADC1_EXTI15/ADC2_EXTI15/TIM1_CH3N)
- net Enc4: now reaches P4.5 (P5)
- net Enc4: now also U6.32 (ADC1_EXTI11/ADC2_EXTI11/CAN_RX/TIM1_CH4/USART1_CTS/USB_DM/PA11)
- net at U10.12 (3A), U10.2 (1A): now also U6.29 (RCC_MCO/TIM1_CH1/USART1_CK/PA8)
- net at U10.19 (4A), U10.9 (2A): now also U6.30 (TIM1_CH2/USART1_TX/PA9)
- net at U10.1 (1,2EN), U10.11 (3,4_EN): now also U6.31 (TIM1_CH3/USART1_RX/PA10)
- net P11: now reaches P1.1 (P1)
- net P11: now also U6.21 (PB10/TIM2_CH3)
- net at P2.6 (P6): now also U6.41 (PB5/I2C1_SMBA/SPI1_MOSI/TIM3_CH2)
- net at P2.5 (P5): now also U6.42 (PB6/I2C1_SCL/USART1_TX)
- net at P2.4 (P4): now also U6.43 (PB7/I2C1_SDA/USART1_RX)
- net at P2.3 (P3): now also U6.45 (PB8/CAN_RX/I2C1_SCL)
- net at R10.2, R6.1: now also U6.44 (BOOT0)
- net at P2.2 (P2): now also U6.46 (PB9/CAN_TX/I2C1_SDA)
- net P21: now reaches P2.1 (P1)
- net P21: now also U6.40 (PB4/SPI1_MISO/SYS_NJTRST/TIM3_CH1)
- net at C1.2, R5.2, S1.1: now also U6.7 (NRST)
- net at D4.2 (A): now also P6.5 (P5)
- new net SWO: P6.2 (P2), U6.39 (PB3/SPI1_SCK/SYS_JTDO-TRACESWO/TIM2_CH2)
- no-connect marks 10 -> 6
Other:
- moved on the sheet: C15, C16, C17, C19, C21, C3, C4, C5, P2, P3, P4

Commit message: final
Parts:
- removed U2, U3: LTV-358T, Buttons_Switches_SMD:SW_DIP_x2_W6.15mm_Slide_Omron_A6H, symbol LTV-358T-RESCUE-pcb1
- added P7: CONN_01X02, SparkFun:SparkFun-1X02, symbol CONN_01X02
- added U2, U3: TLP291, MyLib:Gul_wings_4, symbol TLP291
- Q1: footprint TO_SOT_Packages_THT:TO-220_Vertical -> TO_SOT_Packages_SMD:SOT-23
Connections:
- net +5C: now also P7.1 (P1)
- net Enc0: no longer U6.10 (ADC1_IN0/ADC2_IN0/SYS_WKUP/TIM2_CH1/TIM2_ETR/USART2_CTS/PA0)
- net Enc1: no longer U6.11 (ADC1_IN1/ADC2_IN1/TIM2_CH2/USART2_RTS/PA1)
- net GND: now also P7.2 (P2), U2.3, U3.2
- net VSS: now also U2.2, U3.3
- net at R9.2: now also U2.4
- net at R7.1, U1.2: now also U2.1
- net at R1.1: now also U3.4
- net at R8.1, U5.2: now also U3.1
- no-connect marks 6 -> 8
